Commit message: custom gate heights

File: safe_control_gym/envs/gym_pybullet_drones/assets/low_portal.urdf (robot description, URDF)
Before this commit: robot architrave, 6 links, 5 joints
Links:
- removed link box_link
- added link support, mass 1.0; collision cylinder length=0.05 radius=0.05; visual cylinder length=0.05 radius=0.05
- link base_link: mass 0.1 -> 100; geometry visual sphere radius=100
Joints:
- removed joint box_joint
- added joint support_joint: type fixed, parent base_link, child support

File: safe_control_gym/envs/gym_pybullet_drones/assets/portal.urdf (robot description, URDF)
Before this commit: robot architrave, 6 links, 5 joints
Links:
- link support: geometry collision cylinder length=0.275 radius=0.05; visual cylinder length=0.275 radius=0.05
