Commit message: more work with gate spawning and trajectory generation

File: safe_control_gym/envs/gym_pybullet_drones/assets/obstacle.urdf (robot description, URDF)
Before this commit: robot architrave, 2 links, 1 joints
Links:
- link base_link: geometry collision cylinder length=1 radius=0.05; visual cylinder length=1 radius=0.05
